File: 4ch-relay-1fan-pcb.kicad_pcb (KiCad board)
At the start: 2 copper layers, 54 parts, among them J1 Screw_Terminal_01x03, J2 Conn_01x06_Pin, J3 Screw_Terminal_01x03, J4 Screw_Terminal_01x03, J5 Screw_Terminal_01x03, J7 Conn_01x02, K1 Relay_SPDT, K2 Relay_SPDT, K3 Relay_SPDT, K4 Relay_SPDT, Q1 2N3904, Q2 2N3904, Q3 2N3904, Q4 2N3904, Q5 BT136, U1 PC817, U2 PC817, U3 PC817, U4 PC817, U5 MOC3021M, U6 PC817

Commit message: Add files via upload
Parts:
- moved D1 56.2 mm to (175.8, 114.5)
- moved D2 56.2 mm to (175.1, 95.7)
- moved D4 56.2 mm to (151.9, 95.7)
- moved D6 56.2 mm to (128.6, 95.7)
- moved Q1 56.2 mm to (166.9, 102.0)
- moved Q2 56.2 mm to (143.7, 102.0)
- moved R4 56.2 mm to (161.2, 118.2)
- moved R5 56.2 mm to (138.5, 118.2)
- moved BR1 56.2 mm to (201.3, 87.3)
- moved C1 56.2 mm to (192.1, 93.5)
- moved D3 56.2 mm to (153.1, 114.2)
- moved J3 56.2 mm to (151.6, 68.0)
- moved J4 56.2 mm to (128.7, 68.1)
- moved J6 56.2 mm to (203.8, 67.3)
- moved J7 56.2 mm to (139.7, 128.1)
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