File: 4ch-relay-1fan-pcb.kicad_pcb (KiCad board)
At the start: 2 copper layers, 54 parts, among them J1 Screw_Terminal_01x03, J2 Conn_01x06_Pin, J3 Screw_Terminal_01x03, J4 Screw_Terminal_01x03, J5 Screw_Terminal_01x03, J7 Conn_01x02, K1 Relay_SPDT, K2 Relay_SPDT, K3 Relay_SPDT, K4 Relay_SPDT, Q1 2N3904, Q2 2N3904, Q3 2N3904, Q4 2N3904, Q5 BT136, U1 PC817, U2 PC817, U3 PC817, U4 PC817, U5 MOC3021M, U6 PC817

Commit message: Add files via upload
Parts:
- removed J7: Conn_01x02, Connector_PinHeader_2.54mm:PinHeader_1x02_P2.54mm_Vertical
- J2: value Conn_01x06_Pin -> Conn_01x08_Pin; footprint Connector_PinHeader_2.54mm:PinHeader_1x06_P2.54mm_Vertical -> Connector_PinHeader_2.54mm:PinHeader_1x08_P2.54mm_Vertical
- moved J2 5.31 mm to (142.2, 129.4)
Connections:
- J2 pad 5: GND -> Net-(J2-Pin_5)
- J2 pad 6: +5V -> Net-(J2-Pin_6)
- R13 pad 1: Net-(J2-Pin_4) -> Net-(J2-Pin_6)
- R17 pad 2: Net-(J7-Pin_2) -> Net-(J2-Pin_1)
- R21 pad 2: Net-(J7-Pin_1) -> Net-(J2-Pin_2)
- R4 pad 1: Net-(J2-Pin_1) -> Net-(J2-Pin_3)
- R5 pad 1: Net-(J2-Pin_2) -> Net-(J2-Pin_4)
- R9 pad 1: Net-(J2-Pin_3) -> Net-(J2-Pin_5)
- U6 pad 4: Net-(J7-Pin_1) -> Net-(J2-Pin_2)
Routing:
- net Net-(J7-Pin_1): track 95.5 -> 0.00 mm
- net Net-(J2-Pin_2): track 12.4 -> 96.8 mm
- net Net-(J7-Pin_2): track 50.8 -> 0.00 mm
- net Net-(J2-Pin_6): track 0.00 -> 46.1 mm
- net Net-(J2-Pin_4): track 44.7 -> 13.5 mm
- net Net-(J2-Pin_5): track 0.00 -> 25.5 mm
- net Net-(J2-Pin_1): track 31.6 -> 52.1 mm
- net Net-(J2-Pin_3): track 24.1 -> 32.7 mm
- net GND: track 200.4 -> 201.8 mm
- net +5V: track 219.1 -> 220.5 mm

Commit message: Add files via upload
Routing:
- net Net-(J6-Pin_1): track 14.8 -> 45.0 mm
Changed lines of the file:
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@@
+	)
+	(segment
+		(start 195.47 86.92)
+		(end 205.43 86.92)
+		(width 2)
+		(layer "B.Cu")
+		(net "Net-(J6-Pin_1)")
+	)
+	(segment
+		(start 205.325 74.445)
+		(end 203.81 74.445)
+		(width 2)
+		(layer "B.Cu")
+		(net "Net-(J6-Pin_1)")
 	)
 	(segment
@@
 		(width 2)
 		(layer "B.Cu")
+		(net "Net-(J6-Pin_1)")
+	)
+	(segment
+		(start 207.16 76.28)
+		(end 205.325 74.445)
+		(width 2)
+		(layer "B.Cu")
+		(net "Net-(J6-Pin_1)")
+	)
+	(segment
+		(start 207.16 85.19)
+		(end 207.16 76.28)
+		(width 2)
+		(layer "B.Cu")
+		(net "Net-(J6-Pin_1)")
+	)
+	(segment
+		(start 192.06 83.51)
+		(end 195.47 86.92)
+		(width 2)
+		(layer "B.Cu")
+		(net "Net-(J6-Pin_1)")
+	)
+	(segment
+		(start 205.43 86.92)
+		(end 207.16 85.19)
+		(width 2)
+		(layer "B.Cu")

Commit message: Add files via upload
Other:
- board text added: "5v"
- board text added: "Gnd"
- board text added: "R1"
- board text added: "R2"
- board text added: "R3"
- board text added: "R4"
- board text added: "TRI"
- board text added: "ZCD"
