File: 4ch-relay-1fan-pcb.kicad_pcb (KiCad board)
At the start: 2 copper layers, 53 parts, among them J1 Screw_Terminal_01x03, J2 Conn_01x08_Pin, J3 Screw_Terminal_01x03, J4 Screw_Terminal_01x03, J5 Screw_Terminal_01x03, K1 Relay_SPDT, K2 Relay_SPDT, K3 Relay_SPDT, K4 Relay_SPDT, Q1 2N3904, Q2 2N3904, Q3 2N3904, Q4 2N3904, Q5 BT136, U1 PC817, U2 PC817, U3 PC817, U4 PC817, U5 MOC3021M, U6 PC817

Commit message: Add files via upload
Routing:
- net Net-(J2-Pin_5): track 25.5 -> 26.4 mm
Changed lines of the file:
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@@
 	)
 	(segment
-		(start 132.09 123.43)
+		(start 115.0675 118.805)
+		(end 116.8175 120.555)
+		(width 1)
+		(layer "B.Cu")
+		(net "Net-(J2-Pin_5)")
+	)
+	(segment
+		(start 132.09 121.8)
 		(end 132.09 129.38)
 		(width 1)
@@
 	)
 	(segment
-		(start 129.215 120.555)
-		(end 132.09 123.43)
+		(start 116.8175 120.555)
+		(end 130.845 120.555)
 		(width 1)
 		(layer "B.Cu")
@@
 	)
 	(segment
-		(start 116.8175 120.555)
-		(end 129.215 120.555)
+		(start 130.845 120.555)
+		(end 132.09 121.8)
 		(width 1)
 		(layer "B.Cu")
@@
 		(width 1)
 		(layer "B.Cu")
-		(net "Net-(J2-Pin_5)")
-	)
-	(segment
-		(start 115.0675 118.805)
-		(end 116.8175 120.555)
-		(width 1)
-		(layer "B.Cu")

Commit message: Add files via upload
Other:
- board outline added: 127.6 x 76.4 mm
- board text added: "CO"
- board text added: "Fan"
- board text added: "L"
- board text added: "N"
- board text added: "NC"
- board text added: "NO"
Changed lines of the file:
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@@
 			(at 2.5 5 0)
 			(layer "F.SilkS")
+			(hide yes)
 			(effects
 				(font
@@
 		)
 		(property "Value" "~"
-			(at 2.25 4.92 0)
+			(at 2.36 4.76 0)
 			(layer "F.Fab")
 			(effects
@@
 			(at 2 5 0)
 			(layer "F.SilkS")
+			(hide yes)
 			(effects
 				(font
@@
 		)
 		(property "Value" "~"
-			(at -11.4125 8.3075 90)
+			(at 2.46 4.76 0)
 			(layer "F.Fab")
 			(effects
@@
 		(layer "F.SilkS")
 	)
+	(gr_rect
+		(start 85.74 58.72)
+		(end 213.34 135.14)
+		(stroke
+			(width 0.05)
+			(type default)
+		)
+		(fill no)
+		(layer "Edge.Cuts")
+	)
 	(gr_text "SASoftwareS"
 		(at 202 126 0)
@@
 		)
 	)
+	(gr_text "NC"
+		(at 95.7 61.33 90)
+		(layer "F.SilkS")
+		(effects
+			(font
+				(size 0.8 0.8)
+				(thickness 0.1)
+			)
+			(justify left bottom)
+		)
+	)
+	(gr_text "CO"
+		(at 100.92 61.3 90)
+		(layer "F.SilkS")
+		(effects
+			(font
+				(size 0.8 0.8)
+				(thickness 0.1)
+			)
+			(justify left bottom)
+		)
+	)
+	(gr_text "NO"
+		(at 105.77 61.33 90)
+		(layer "F.SilkS")
+		(effects
+			(font
+				(size 0.8 0.8)
+				(thickness 0.1)
+			)
+			(justify left bottom)
+		)
+	)
+	(gr_text "NC"
+		(at 119.04 61.5 90)
+		(layer "F.SilkS")
+		(effects
+			(font
+				(size 0.8 0.8)
+				(thickness 0.1)
+			)
+			(justify left bottom)
+		)
+	)
+	(gr_text "CO"
+		(at 124.26 61.47 90)
+		(layer "F.SilkS")
+		(effects
+			(font
+				(size 0.8 0.8)
+				(thickness 0.1)
+			)
+			(justify left bottom)
+		)
+	)
+	(gr_text "NO"
+		(at 129.11 61.5 90)
+		(layer "F.SilkS")
+		(effects
+			(font
+				(size 0.8 0.8)
+				(thickness 0.1)
+			)
+			(justify left bottom)
+		)
+	)
+	(gr_text "NC"
+		(at 141.79 61.45 90)
+		(layer "F.SilkS")
+		(effects
+			(font
+				(size 0.8 0.8)
+				(thickness 0.1)
+			)
+			(justify left bottom)
+		)
+	)
+	(gr_text "CO"
+		(at 147.01 61.42 90)
+		(layer "F.SilkS")
+		(effects
+			(font
+				(size 0.8 0.8)
+				(thickness 0.1)
+			)
+			(justify left bottom)
+		)
+	)
+	(gr_text "NO"
+		(at 151.86 61.45 90)
+		(layer "F.SilkS")
+		(effects
+			(font
+				(size 0.8 0.8)
+				(thickness 0.1)
+			)
+			(justify left bottom)
+		)
+	)
+	(gr_text "NC"
+		(at 165.13 61.48 90)
+		(layer "F.SilkS")
+		(effects
+			(font
+				(size 0.8 0.8)
+				(thickness 0.1)
+			)
+			(justify left bottom)
+		)
+	)
+	(gr_text "CO"
+		(at 170.35 61.45 90)
+		(layer "F.SilkS")
+		(effects
+			(font
+				(size 0.8 0.8)
+				(thickness 0.1)
+			)
+			(justify left bottom)
+		)
+	)
+	(gr_text "NO"
+		(at 175.2 61.48 90)
+		(layer "F.SilkS")
+		(effects
+			(font
+				(size 0.8 0.8)
+				(thickness 0.1)
+			)
+			(justify left bottom)
+		)
+	)
+	(gr_text "Fan"
+		(at 187.42 61.94 90)
+		(layer "F.SilkS")
+		(effects
+			(font
+				(size 0.8 0.8)
+				(thickness 0.1)
+			)
+			(justify left bottom)
+		)
+	)
+	(gr_text "N"
+		(at 192.5 61.21 90)
+		(layer "F.SilkS")
+		(effects
+			(font
+				(size 0.8 0.8)
+				(thickness 0.1)
+			)
+			(justify left bottom)
+		)
+	)
+	(gr_text "N"
+		(at 199.32 61.18 90)
+		(layer "F.SilkS")
+		(effects
+			(font
+				(size 0.8 0.8)
+				(thickness 0.1)
+			)
+			(justify left bottom)
+		)
+	)
+	(gr_text "L"
+		(at 204.14 61.04 90)
+		(layer "F.SilkS")
+		(effects
+			(font
+				(size 0.8 0.8)
+				(thickness 0.1)
+			)
+			(justify left bottom)
+		)
+	)

Commit message: Add files via upload
Parts:
- added ?: , , F.Cu at (210.2, 132.0)
- added ?: , , F.Cu at (88.9, 61.9)
- added ?: , , F.Cu at (89.0, 131.9)
- added ?: , , F.Cu at (210.1, 62.0)
Other:
- board text added: "5v G R1 R2 R3 R4 ZC T"
- board text removed: "5v"
- board text removed: "Gnd"
- board text removed: "R1"
- board text removed: "R2"
- board text removed: "R3"
- board text removed: "R4"
- board text removed: "TRI"
- board text removed: "ZCD"
