File: 4ch-relay-1fan-pcb.kicad_sch (KiCad schematic)
At the start: 54 parts, among them J1 Screw_Terminal_01x03, J2 Conn_01x06_Pin, J3 Screw_Terminal_01x03, J4 Screw_Terminal_01x03, J5 Screw_Terminal_01x03, J7 Conn_01x02, K1 Relay_SPDT, K2 Relay_SPDT, K3 Relay_SPDT, K4 Relay_SPDT, Q1 2N3904, Q2 2N3904, Q3 2N3904, Q4 2N3904, Q5 BT136, U1 PC817, U2 PC817, U3 PC817, U4 PC817, U5 MOC3021M, U6 PC817

Commit message: Add files via upload
Parts:
- removed J2: Conn_01x06_Pin, Connector_PinHeader_2.54mm:PinHeader_1x06_P2.54mm_Vertical, symbol Connector:Conn_01x06_Pin
- removed J7: Conn_01x02, Connector_PinHeader_2.54mm:PinHeader_1x02_P2.54mm_Vertical, symbol Connector_Generic:Conn_01x02
- added J2: Conn_01x08_Pin, Connector_PinHeader_2.54mm:PinHeader_1x08_P2.54mm_Vertical, symbol Connector:Conn_01x08_Pin
Connections:
- net +5V: now also J2.8 (Pin_8)
- net GND: now also J2.7 (Pin_7)
- net at R4.1: now also J2.3 (Pin_3)
- net at R21.2, U6.4: now also J2.2 (Pin_2)
- net at R17.2: now also J2.1 (Pin_1)
- net at R5.1: now also J2.4 (Pin_4)
- net at R9.1: now also J2.5 (Pin_5)
- net at R13.1: now also J2.6 (Pin_6)
Other:
- moved on the sheet: BR1, C1, D1, D2, D3, D4, D5, D6, D7, D8, J1, J3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
